Commit message: added naive motion controller

File: src/add_post_pro2/depowdering_aman/urdf/depowdering_gripper_robot.xacro (robot description, xacro)
@@ -1,6 +1,6 @@
 <?xml version="1.0"?>
 <robot xmlns:xacro="http://ros.org/wiki/xacro" name="add_post_pro_depowdering">
-  <!-- Include the robot xacro file -->
-  <xacro:include filename="$(find denso_robot_descriptions)/vs6577_description/urdf/vs6577.transmission.xacro"/>
+	<!-- Include the robot xacro file -->
+	<xacro:include filename="$(find denso_robot_descriptions)/vs6577_description/urdf/vs6577.transmission.xacro"/>
 	<gazebo>
         <plugin filename="libgazebo_ros_control.so" name="gazebo_ros_control">
@@ -151,20 +151,20 @@
 	</gazebo>
 	<gazebo reference="J1">
-		<material>Gazebo/Gray</material>
+		<material>Gazebo/White</material>
 	</gazebo>
 	<gazebo reference="J2">
-		<material>Gazebo/Gray</material>
+		<material>Gazebo/White</material>
 	</gazebo>
 	<gazebo reference="J3">
-		<material>Gazebo/Gray</material>
+		<material>Gazebo/White</material>
 	</gazebo>
 	<gazebo reference="J4">
-		<material>Gazebo/Gray</material>
+		<material>Gazebo/White</material>
 	</gazebo>
 	<gazebo reference="J5">
-		<material>Gazebo/Gray</material>
+		<material>Gazebo/White</material>
 	</gazebo>
 	<gazebo reference="J6">
-		<material>Gazebo/Gray</material>
+		<material>Gazebo/White</material>
 	</gazebo>
 	<gazebo>
@@ -279,5 +279,5 @@
 		<origin xyz="0 0 0.004" rpy="0 0 3.14" />
 		<parent link="J6" />
-		<child  link="gripper_base_link" />
+		<child link="gripper_base_link" />
 		<axis xyz="0 0 -1" />
 	</joint>
@@ -287,6 +287,12 @@
 		<child link="gripper_Link" />
 		<axis xyz="0 0 -1" />
-		<limit lower="0" upper="0.021" effort="0" velocity="0" />
-	</joint>
+		<limit lower="0" upper="0.021" effort="1" velocity="1" />
+	</joint>
+	<gazebo reference="gripper_base_link">
+		<material>Gazebo/Gray</material>
+	</gazebo>
+	<gazebo reference="gripper_Link">
+		<material>Gazebo/Gray</material>
+	</gazebo>
 	<!--########### adding transmissions ########### -->
 	<!-- <transmission
@@ -301,12 +307,11 @@
 		</actuator>
 	</transmission> -->
-	<transmission
-		name="trans_gripper">
+	<transmission name="trans_gripper">
 		<type>transmission_interface/SimpleTransmission</type>
 		<joint name="gripper_Joint">
-			<hardwareInterface>hardware_interface/PositionJointInterface</hardwareInterface>
+			<hardwareInterface>hardware_interface/EffortJointInterface</hardwareInterface>
 		</joint>
 		<actuator name="motor_gripper">
-			<hardwareInterface>hardware_interface/PositionJointInterface</hardwareInterface>
+			<hardwareInterface>hardware_interface/EffortJointInterface</hardwareInterface>
 			<mechanicalReduction>1</mechanicalReduction>
 		</actuator>

Commit message: gazebo movement

File: src/add_post_pro2/depowdering_aman/urdf/depowdering_gripper_robot.xacro (robot description, xacro)
@@ -269,10 +269,10 @@
 			</material>
 		</visual>
-		<collision>
+		<!-- <collision>
 			<origin xyz="0 0 0" rpy="0 0 0" />
 			<geometry>
 				<mesh filename="package://add_post_pro_simulation/mesh/gripper_Link.STL" />
 			</geometry>
-		</collision>
+		</collision> -->
 	</link>
 	<joint name="gripper_base_Joint" type="fixed">

File: src/add_post_pro_gripper_config/config/gazebo_add_post_pro_depowdering.urdf (robot description, URDF)
Before this commit: robot add_post_pro_depowdering, 10 links, 9 joints
Links:
- link gripper_Link: geometry visual mesh filename=package://add_post_pro_simulation/mesh/gripper_Link.STL
